File: compactActiveLoad.sch (KiCad schematic (older format))
At the start: 10 parts, among them CON1 Keystone_3002, CON2 Keystone_3002, CON3 LOAD, CON4 +12V, CON5 MOD, Q1 IRLR024NPBF, Q2 IRLR024NPBF, SW1 SW_1290F1123, SW2 SW_1290F1123, U1 Heatsink_55mm_CG128

Commit message: Placement
Parts:
- added C1: N.C., pnRLC:0603, symbol C
- added C2: 100n, 0603, symbol C
- added C3, C4: 100n, 0805, symbol C
- added CON6: FAN, pnConnector:PAD2_2x3, symbol CON2
- added P1: 10k, pnRLC:pot_ACP_CA6VSMD+6001, symbol pot_ACP_CA6VSMD+6001
- added R1, R8: 1k, pnRLC:0603, symbol R
- added R2: 100R, pnRLC:0603, symbol R
- added R3, R4, R5, R6: 1R, pnRLC:R2010, symbol R
- added R7: 10k, pnRLC:0603, symbol R
- added U1: LMV116MF, SOT23-5, symbol LMV116MF
- added U2: LP2981A-50DBVR, pnSemiconductor:SOT23-5, symbol LP2981A-50DBVR
- renumbered U1 to HS1
Connections:
- net at Q1.1 (G): now also Q2.1 (G), R2.1
- net at Q1.3 (S): now also R3.2, R4.2, R8.1
- net Load: now reaches Q1.4 (D)
- net Load: now also CON3.2, HS1.HS, Q2.4 (D)
- net at Q2.3 (S): now also R1.1, R5.2, R6.2
- net Vbat: now reaches CON1.+
- net Vbat: now also SW1.NC
- net at CON1.-: now also CON2.+
- net GND: now reaches CON2.-
- net GND: now also CON3.1, CON4.1, CON5.1, HS1.MNT, SW1.MNT, SW2.MNT, C2.2, C3.2, C4.2, CON6.2, P1.1, R3.1, R4.1, R5.1, R6.1, R7.1, U1.2 (VSS), U2.2 (GND)
- net VCC: now reaches SW1.COM
- net VCC: now also C2.1, P1.3, U1.5 (VDD)
- net +5V: now reaches SW1.NO
- net +5V: now also C4.1, U2.5 (OUT)
- net Vin: now reaches SW2.COM
- net Vin: now also R7.2, U1.3 (+)
- net at SW2.NC: now also P1.2
- net at SW2.NO: now also CON5.2
- net +12V: now reaches CON4.2
- net +12V: now also C3.1, CON6.1, U2.1 (IN), U2.3 (EN)
- new net Vfb: C1.2, R1.2, R8.2, U1.4 (-)
- new net Vout: C1.1, R2.2, U1.1 (OUT)
Other:
- moved on the sheet: CON1, CON2, CON3, CON4, CON5, HS1, Q1, Q2, SW1, SW2

Commit message: routing
Parts:
- removed C4: 100n, 0805, symbol C
- added C4: TAJA106M010RNJ, pnRLC:TANTAL_A, symbol Cpol
- added C5: 10n, R0603, symbol C
- added R9: 10k, R0603, symbol R
- C1, R1, R2, R7, R8: footprint pnRLC:0603 -> R0603
- C2: footprint 0603 -> R0603
- C3: value 100n -> 2u2u/25V; footprint 0805 -> R0805
- P1: value 10k -> 1k
Connections:
- net +5V: now also C4.1
- net GND: now also C4.2, C5.2
- net VCC: now also R9.2; no longer P1.3
- net at CON5.2, SW2.NO: now also C5.1
- new net: P1.3, R9.1
Other:
- moved on the sheet: C1, C2, CON5, P1, R7, SW2, U1

Commit message: Routed
Parts:
- added TP1, TP4, TP7: GND, pnConnector:TP_1mm, symbol Testpoint
- added TP2: Vin, pnConnector:TP_1mm, symbol Testpoint
- added TP5: Vout, pnConnector:TP_1mm, symbol Testpoint
- added TP6: Vfb, pnConnector:TP_1mm, symbol Testpoint
- added TP8: Load, pnConnector:TP_1mm, symbol Testpoint
- SW1: value SW_1290F1123 -> Bat/Ext
- SW2: value SW_1290F1123 -> Ext/Int
Connections:
- net GND: now also TP1.1, TP4.1, TP7.1
- net Load: now also TP8.1
- net Vfb: now also TP6.1
- net Vin: now also TP2.1
- net Vout: now also TP5.1
Changed lines of the file:
@@
 	4950 1100 4500 1100
-Wire Wire Line
-	4500 1100 4500 1300
 Wire Wire Line
 	4500 1500 4500 1600
@@
 P 4400 4100
 F 0 "SW2" H 4400 4300 60  0000 C CNN
-F 1 "SW_1290F1123" H 4400 3950 40  0001 C CNN
+F 1 "Ext/Int" H 4600 3900 40  0000 C CNN
 F 2 "SW_1290F1123" H 4400 3900 40  0001 C CNN
 F 3 "" H 4400 4100 60  0000 C CNN
@@
 P 5300 1000
 F 0 "SW1" H 5300 1200 60  0000 C CNN
-F 1 "SW_1290F1123" H 5300 850 40  0001 C CNN
+F 1 "Bat/Ext" H 5500 800 40  0000 C CNN
 F 2 "SW_1290F1123" H 5300 800 40  0001 C CNN
 F 3 "" H 5300 1000 60  0000 C CNN
@@
 	1    0    0    -1
 $EndComp
+$Comp
+L Testpoint TP2
+U 1 1 55852A5A
+P 4450 3600
+F 0 "TP2" H 4500 3650 60  0000 L CNN
+F 1 "Vin" H 4500 3550 60  0000 L CNN
+F 2 "pnConnector:TP_1mm" H 4450 3600 60  0001 C CNN
+F 3 "" H 4450 3600 60  0000 C CNN
+	1    4450 3600
+	1    0    0    -1
+$EndComp
+Wire Wire Line
+	4450 3650 4450 3700
+Connection ~ 4450 3700
+$Comp
+L Testpoint TP5
+U 1 1 55852F33
+P 6550 3700
+F 0 "TP5" H 6600 3750 60  0000 L CNN
+F 1 "Vout" H 6600 3650 60  0000 L CNN
+F 2 "pnConnector:TP_1mm" H 6550 3700 60  0001 C CNN
+F 3 "" H 6550 3700 60  0000 C CNN
+	1    6550 3700
+	1    0    0    -1
+$EndComp
+Wire Wire Line
+	6550 3750 6550 3800
+Connection ~ 6550 3800
+$Comp
+L Testpoint TP6
+U 1 1 55853027
+P 6550 4350
+F 0 "TP6" H 6600 4400 60  0000 L CNN
+F 1 "Vfb" H 6600 4300 60  0000 L CNN
+F 2 "pnConnector:TP_1mm" H 6550 4350 60  0001 C CNN
+F 3 "" H 6550 4350 60  0000 C CNN
+	1    6550 4350
+	-1   0    0    1
+$EndComp
+Wire Wire Line
+	6550 4300 6550 4250
+Connection ~ 6550 4250
+$Comp
+L Testpoint TP8
+U 1 1 55853377
+P 8900 3350
+F 0 "TP8" H 8950 3400 60  0000 L CNN
+F 1 "Load" H 8950 3300 60  0000 L CNN
+F 2 "pnConnector:TP_1mm" H 8900 3350 60  0001 C CNN
+F 3 "" H 8900 3350 60  0000 C CNN
+	1    8900 3350
+	1    0    0    -1
+$EndComp
+Wire Wire Line
+	8900 3400 8900 3450
+Connection ~ 8900 3450
+$Comp
+L GND #PWR021
+U 1 1 558535CF
+P 5900 5000
+F 0 "#PWR021" H 5900 4750 50  0001 C CNN
+F 1 "GND" H 5900 4850 50  0000 C CNN
+F 2 "" H 5900 5000 60  0000 C CNN
+F 3 "" H 5900 5000 60  0000 C CNN
+	1    5900 5000
+	1    0    0    -1
+$EndComp
+$Comp
+L Testpoint TP4
+U 1 1 5585361E
+P 5900 4900
+F 0 "TP4" H 5950 4950 60  0000 L CNN
+F 1 "GND" H 5950 4850 60  0000 L CNN
+F 2 "pnConnector:TP_1mm" H 5900 4900 60  0001 C CNN
+F 3 "" H 5900 4900 60  0000 C CNN
+	1    5900 4900
+	1    0    0    -1
+$EndComp
+Wire Wire Line
+	5900 4950 5900 5000
+$Comp
+L GND #PWR022
+U 1 1 55853741
+P 6550 5000
+F 0 "#PWR022" H 6550 4750 50  0001 C CNN
+F 1 "GND" H 6550 4850 50  0000 C CNN
+F 2 "" H 6550 5000 60  0000 C CNN
+F 3 "" H 6550 5000 60  0000 C CNN
+	1    6550 5000
+	1    0    0    -1
+$EndComp
+$Comp
+L Testpoint TP7
+U 1 1 55853747
+P 6550 4900
+F 0 "TP7" H 6600 4950 60  0000 L CNN
+F 1 "GND" H 6600 4850 60  0000 L CNN
+F 2 "pnConnector:TP_1mm" H 6550 4900 60  0001 C CNN
+F 3 "" H 6550 4900 60  0000 C CNN
+	1    6550 4900
+	1    0    0    -1
+$EndComp
+Wire Wire Line
+	6550 4950 6550 5000
+Wire Wire Line
+	4500 1100 4500 1300
+$Comp
+L GND #PWR023
+U 1 1 55854244
+P 7250 5000
+F 0 "#PWR023" H 7250 4750 50  0001 C CNN
+F 1 "GND" H 7250 4850 50  0000 C CNN
+F 2 "" H 7250 5000 60  0000 C CNN
+F 3 "" H 7250 5000 60  0000 C CNN
+	1    7250 5000
+	1    0    0    -1
+$EndComp
+$Comp
+L Testpoint TP1
+U 1 1 5585424A
+P 7250 4900
+F 0 "TP1" H 7300 4950 60  0000 L CNN
+F 1 "GND" H 7300 4850 60  0000 L CNN
+F 2 "pnConnector:TP_1mm" H 7250 4900 60  0001 C CNN
+F 3 "" H 7250 4900 60  0000 C CNN
+	1    7250 4900
+	1    0    0    -1
+$EndComp
+Wire Wire Line
+	7250 4950 7250 5000
 $EndSCHEMATC

Commit message: Some changes
Other:
- note added: "Add serial resistor (ESD)"
- moved on the sheet: C5, CON5, P1, R7, R9, SW2, TP2
